File: mu.kicad_sch (KiCad schematic)
At the start: 71 parts, among them J1 USB_C_Receptacle_USB2.0_16P, J2 Conn_02x03_Odd_Even, J4 2060-1452/998-404, J5 ESQ-110-X-X-D, U1 STM32F042F6P6, U10 TLV3603QDCKRQ1, U11 SN74LVC1G74DCUT, U12 LM4040AIM3-2.5/NOPB, U13 MCP4921-E/SN, U14 BMP390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

Commit message: nearly done now
Connections:
- net CAN_rx is gone; now on net CAN_-: U9.4 (R)
- net CAN_rx- is gone; now on net CAN_-: J2.1 (Pin_1)
- net CAN_tx is gone; now on net CAN_+: U9.1 (D)
- net CAN_tx+ is gone; now on net CAN_+: J2.2 (Pin_2)
- net PA11- is gone; now on net PA-: J2.3 (Pin_3)
- net PA12+ is gone; now on net PA+: J2.4 (Pin_4)
- net CAN_+: no longer D3.1 (K), R14.1, U9.7 (CANH)
- net CAN_-: no longer D3.2 (K), R14.2, U9.6 (CANL)
- net GND: no longer U3.1
- net at R3.2, U6.3 (NONIINVERTINGINPUT): now also U3.1; no longer U3.2
- net CAN_hi renamed CAN_o+
- net CAN_o+: now also D3.1 (K), R14.1, U9.7 (CANH)
- net CAN_lo renamed CAN_o-
- net CAN_o-: now also D3.2 (K), R14.2, U9.6 (CANL)
- net PA11 renamed PA-
- net PA12 renamed PA+
- no-connect marks 12 -> 13
Other:
- note added: "pa11 is pa- pa12 is pa+"
- note added: "rx is + tx is -"
- note removed: "fast output"
- moved on the sheet: C1, C2, C3, U3

Commit message: restructuring now that we've got the standard connector
Parts:
- added C31: 47uF, Capacitor_SMD:C_0402_1005Metric, symbol Device:C
- added R17: 60Ω, Resistor_SMD:R_0402_1005Metric, symbol Device:R
- R14: value 120Ω -> 60Ω
Connections:
- net CAN_o+: now also R17.1; no longer R14.1
- net GND: now also C31.2
- new net: C31.1, R14.1, R17.2
Other:
- note added: "-"
- note added: "rxd"
- note added: "this is going up 9km, is the bias voltage ok?"
- note added: "txd"
- note added: "txd rxd"
- note removed: "pa11 is pa- pa12 is pa+"
- note removed: "rx is + tx is -"
- moved on the sheet: C23, C24, D3, R10, R14, U9

Commit message: programming stuff
Parts:
- added J3: Conn_02x03_Odd_Even, Connector_PinHeader_1.00mm:PinHeader_2x03_P1.00mm_Vertical, symbol Connector_Generic:Conn_02x03_Odd_Even
Connections:
- net 3.3V_Dig: now also J3.6 (Pin_6)
- net GND: now also J3.3 (Pin_3), J3.5 (Pin_5)
- net SWCLK: now also J3.4 (Pin_4)
- net SWDIO: now also J3.2 (Pin_2)
- net NRST: now reaches C13.1, R5.1, U1.4 (NRST)
- net NRST: now also J3.1 (Pin_1)
Other:
- moved on the sheet: C13, R5

Commit message: ready to send off to stephen
Connections:
- net 2.5V_Ref: now also U3.1
- net GND: now also J5.13
- net at R3.2, U6.3 (NONIINVERTINGINPUT): now also U3.2; no longer U3.1
- no-connect marks 13 -> 12
Other:
- note removed: "should the be 2.5v?"
- moved on the sheet: C15, C30, J1, J2, R12, R13, R7, R8, U14, U7

Commit message: higher voltage diode
Parts:
- removed D1: BAT54J, Diode_SMD:D_SOD-323F, symbol Diode:BAT54J
- added CR1: BAT46JFILM, SOD-323_STM, symbol BAT46J:BAT46JFILM
Connections:
- net at C4.1, R1.2, R4.2: now also CR1.2
- net at L1.2, U2.6 (LX): now also CR1.1
Changed lines of the file:
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@@
 	(wire
 		(pts
-			(xy 81.28 43.18) (xy 81.28 46.99)
-		)
-		(stroke
-			(width 0)
-			(type default)
-		)
-	)
-	(wire
-		(pts
 			(xy 128.27 81.28) (xy 128.27 82.55)
 		)
@@
 	(wire
 		(pts
+			(xy 81.28 43.18) (xy 81.28 45.72)
+		)
+		(stroke
+			(width 0)
+			(type default)
+		)
+	)
+	(wire
+		(pts
 			(xy 326.39 124.46) (xy 322.58 124.46)
 		)
@@
 	(wire
 		(pts
-			(xy 81.28 54.61) (xy 81.28 62.23)
+			(xy 81.28 55.88) (xy 81.28 62.23)
 		)
 		(stroke
@@
 	)
 	(symbol
+		(lib_id "BAT46J:BAT46JFILM")
+		(at 81.28 55.88 90)
+		(unit 1)
+		(exclude_from_sim no)
+		(in_bom yes)
+		(on_board yes)
+		(dnp no)
+		(property "Reference" "CR1"
+			(at 86.614 48.514 0)
+			(effects
+				(font
+					(size 1.524 1.524)
+				)
+				(justify right)
+			)
+		)
+		(property "Value" "BAT46JFILM"
+			(at 84.582 43.688 0)
+			(effects
+				(font
+					(size 1.524 1.524)
+				)
+				(justify right)
+			)
+		)
+		(property "Footprint" "SOD-323_STM"
+			(at 81.28 55.88 0)
+			(effects
+				(font
+					(size 1.27 1.27)
+					(italic yes)
+				)
+				(hide yes)
+			)
+		)
+		(property "Datasheet" "https://www.st.com/resource/en/datasheet/bat46.pdf"
+			(at 81.28 55.88 0)
+			(effects
+				(font
+					(size 1.27 1.27)
+					(italic yes)
+				)
+				(hide yes)
+			)
+		)
+		(property "Description" ""
+			(at 81.28 55.88 0)
+			(effects
+				(font
+					(size 1.27 1.27)
+				)
+				(hide yes)
+			)
+		)
+		(pin "2"
+		)
+		(pin "1"
+		)
+		(instances
+			(project ""
+				(path "/0020f91a-50ae-478d-8303-55d8991d2d34"
+					(reference "CR1")
+					(unit 1)
+				)
+			)
+		)
+	)
+	(symbol
 		(lib_id "power:GND")
 		(at 232.41 118.11 90)
@@
 					(unit 1)
 				)
-			)
-		)
-	)
-	(symbol
-		(lib_id "Diode:BAT54J")
-		(at 81.28 50.8 270)
-		(unit 1)
-		(exclude_from_sim no)
-		(in_bom yes)
-		(on_board yes)
-		(dnp no)
-		(fields_autoplaced yes)
-		(property "Reference" "D1"
-			(at 83.82 49.2124 90)
-			(effects
-				(font
-					(size 1.27 1.27)
-				)
-				(justify left)
-			)
-		)
-		(property "Value" "BAT54J"
-			(at 83.82 51.7524 90)
-			(effects
-				(font
-					(size 1.27 1.27)
-				)
-				(justify left)
-			)
-		)
-		(property "Footprint" "Diode_SMD:D_SOD-323F"
-			(at 76.835 50.8 0)
-			(effects
-				(font
-					(size 1.27 1.27)
-				)
-				(hide yes)
-			)
-		)
-		(property "Datasheet" "https://assets.nexperia.com/documents/data-sheet/BAT54J.pdf"
-			(at 81.28 50.8 0)
-			(effects
-				(font
-					(size 1.27 1.27)
-				)
-				(hide yes)
-			)
-		)
-		(property "Description" "30V 200mA Schottky diode, SOD-323F"
-			(at 81.28 50.8 0)
-			(effects
-				(font
-					(size 1.27 1.27)
-				)
-				(hide yes)
-			)
-		)
-		(pin "1"
-		)
-		(pin "2"
-		)
-		(instances
-			(project ""
-				(path "/0020f91a-50ae-478d-8303-55d8991d2d34"
-					(reference "D1")
-					(unit 1)
-				)

Commit message: ready to rock and roll
Parts:
- added MOSFET1: IPP80P03P4L04AKSA1, PG-TO220-3-1_INF, symbol IPP80P03P4L04AKSA1:IPP80P03P4L04AKSA1
Connections:
- net GND: now also MOSFET1.1 (G)
- net VBAT_Local: now also MOSFET1.3 (S); no longer J4.1 (1_1), J4.2 (1_2)
- new net: J4.1 (1_1), J4.2 (1_2), MOSFET1.2 (D)
Other:
- moved on the sheet: J4
Changed lines of the file:
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@@
 	(rectangle
 		(start 273.304 162.56)
-		(end 367.284 204.47)
+		(end 399.542 204.47)
 		(stroke
 			(width 0)
@@
 	)
 	(junction
+		(at 356.87 176.53)
+		(diameter 0)
+		(color 0 0 0 0)
+	)
+	(junction
 		(at 256.54 110.49)
 		(diameter 0)
@@
 	)
 	(junction
+		(at 356.87 184.15)
+		(diameter 0)
+		(color 0 0 0 0)
+	)
+	(junction
 		(at 172.72 238.76)
 		(diameter 0)
@@
 	)
 	(junction
-		(at 347.98 181.61)
-		(diameter 0)
-		(color 0 0 0 0)
-	)
-	(junction
 		(at 212.09 167.64)
 		(diameter 0)
@@
 	(wire
 		(pts
+			(xy 347.98 184.15) (xy 356.87 184.15)
+		)
+		(stroke
+			(width 0)
+			(type default)
+		)
+	)
+	(wire
+		(pts
 			(xy 231.14 181.61) (xy 231.14 191.77)
 		)
@@
 	(wire
 		(pts
+			(xy 356.87 176.53) (xy 356.87 179.07)
+		)
+		(stroke
+			(width 0)
+			(type default)
+		)
+	)
+	(wire
+		(pts
 			(xy 224.79 215.9) (xy 224.79 220.98)
 		)
@@
 	(wire
 		(pts
-			(xy 347.98 181.61) (xy 347.98 184.15)
-		)
-		(stroke
-			(width 0)
-			(type default)
-		)
-	)
-	(wire
-		(pts
 			(xy 205.74 73.66) (xy 203.2 73.66)
 		)
@@
 	(wire
 		(pts
+			(xy 356.87 181.61) (xy 356.87 184.15)
+		)
+		(stroke
+			(width 0)
+			(type default)
+		)
+	)
+	(wire
+		(pts
 			(xy 76.2 119.38) (xy 76.2 110.49)
 		)
@@
 	(wire
 		(pts
-			(xy 347.98 176.53) (xy 347.98 179.07)
-		)
-		(stroke
-			(width 0)
-			(type default)
-		)
-	)
-	(wire
-		(pts
 			(xy 248.92 191.77) (xy 252.73 191.77)
 		)
@@
 	(global_label "VBAT_Local"
 		(shape input)
-		(at 347.98 176.53 180)
+		(at 346.71 176.53 180)
 		(fields_autoplaced yes)
 		(effects
@@
 		)
 		(property "Intersheetrefs" "${INTERSHEET_REFS}"
-			(at 334.5325 176.53 0)
+			(at 333.2625 176.53 0)
 			(effects
 				(font
@@
 	(symbol
 		(lib_id "power:GND")
-		(at 347.98 181.61 270)
+		(at 347.98 184.15 270)
 		(unit 1)
 		(exclude_from_sim no)
@@
 		(fields_autoplaced yes)
 		(property "Reference" "#PWR046"
-			(at 341.63 181.61 0)
+			(at 341.63 184.15 0)
 			(effects
 				(font
@@
 		)
 		(property "Value" "GND"
-			(at 344.17 181.6099 90)
+			(at 344.17 184.1499 90)
 			(effects
 				(font
@@
 		)
 		(property "Footprint" ""
-			(at 347.98 181.61 0)
+			(at 347.98 184.15 0)
 			(effects
 				(font
@@
 		)
 		(property "Datasheet" ""
-			(at 347.98 181.61 0)
+			(at 347.98 184.15 0)
 			(effects
 				(font
@@
 		)
 		(property "Description" "Power symbol creates a global label with name \"GND\" , ground"
-			(at 347.98 181.61 0)
+			(at 347.98 184.15 0)
 			(effects
 				(font
@@
 	)
 	(symbol
+		(lib_id "power:GND")
+		(at 351.79 168.91 270)
+		(unit 1)
+		(exclude_from_sim no)
+		(in_bom yes)
+		(on_board yes)
+		(dnp no)
+		(fields_autoplaced yes)
+		(property "Reference" "#PWR053"
+			(at 345.44 168.91 0)
+			(effects
+				(font
+					(size 1.27 1.27)
+				)
+				(hide yes)
+			)
+		)
+		(property "Value" "GND"
+			(at 347.98 168.9099 90)
+			(effects
+				(font
+					(size 1.27 1.27)
+				)
+				(justify right)
+			)
+		)
+		(property "Footprint" ""
+			(at 351.79 168.91 0)
+			(effects
+				(font
+					(size 1.27 1.27)
+				)
+				(hide yes)
+			)
+		)
+		(property "Datasheet" ""
+			(at 351.79 168.91 0)
+			(effects
+				(font
+					(size 1.27 1.27)
+				)
+				(hide yes)
+			)
+		)
+		(property "Description" "Power symbol creates a global label with name \"GND\" , ground"
+			(at 351.79 168.91 0)
+			(effects
+				(font
+					(size 1.27 1.27)
+				)
+				(hide yes)
+			)
+		)
+		(pin "1"
+		)
+		(instances
+			(project "mu"
+				(path "/0020f91a-50ae-478d-8303-55d8991d2d34"
+					(reference "#PWR053")
+					(unit 1)
+				)
+			)
+		)
+	)
+	(symbol
 		(lib_id "Device:R")
 		(at 99.06 43.18 270)
@@
 	)
 	(symbol
+		(lib_id "IPP80P03P4L04AKSA1:IPP80P03P4L04AKSA1")
+		(at 351.79 168.91 270)
+		(unit 1)
+		(exclude_from_sim no)
+		(in_bom yes)
+		(on_board yes)
+		(dnp no)
+		(property "Reference" "MOSFET1"
+			(at 353.568 167.386 90)
+			(effects
+				(font
+					(size 1.524 1.524)
+				)
+				(justify left)
+			)
+		)
+		(property "Value" "IPP80P03P4L04AKSA1"
+			(at 353.568 170.18 90)
+			(effects
+				(font
+					(size 1.524 1.524)
+				)
+				(justify left)
+			)
+		)
+		(property "Footprint" "PG-TO220-3-1_INF"
+			(at 351.79 168.91 0)
+			(effects
+				(font
+					(size 1.27 1.27)
+					(italic yes)
+				)
+				(hide yes)
+			)
+		)
+		(property "Datasheet" "https://www.infineon.com/dgdl/Infineon-I80P03P4L_04-DS-v01_01-en.pdf?fileId=db3a30431ddc9372011e07e95eb827d7"
+			(at 351.79 168.91 0)
+			(effects
+				(font
+					(size 1.27 1.27)
+					(italic yes)
+				)
+				(hide yes)
+			)
+		)
+		(property "Description" ""
+			(at 351.79 168.91 0)
+			(effects
+				(font
+					(size 1.27 1.27)
+				)
+				(hide yes)
+			)
+		)
+		(pin "3"
+		)
+		(pin "2"
+		)
+		(pin "1"
+		)
+		(instances
+			(project ""
+				(path "/0020f91a-50ae-478d-8303-55d8991d2d34"
+					(reference "MOSFET1")
+					(unit 1)
+				)
+			)
+		)
+	)
+	(symbol
 		(lib_id "power:GND")
 		(at 245.11 101.6 270)
@@
 	(symbol
 		(lib_id "Wago_2060-1452 998-404:2060-1452_998-404")
-		(at 347.98 176.53 0)
+		(at 356.87 176.53 0)
 		(unit 1)
 		(exclude_from_sim no)
@@
 		(fields_autoplaced yes)
 		(property "Reference" "J4"
-			(at 361.95 179.0699 0)
+			(at 370.84 179.0699 0)
 			(effects
 				(font
@@
 		)
 		(property "Value" "2060-1452/998-404"
-			(at 361.95 181.6099 0)
+			(at 370.84 181.6099 0)
 			(effects
 				(font
@@
 		)
 		(property "Footprint" "footprints:WAG"
-			(at 347.98 176.53 0)
+			(at 356.87 176.53 0)
 			(effects
 				(font
@@
 		)
 		(property "Datasheet" "2060-1452/998-404"
-			(at 347.98 176.53 0)
+			(at 356.87 176.53 0)
 			(effects
 				(font
@@
 		)
 		(property "Description" ""
-			(at 347.98 176.53 0)
+			(at 356.87 176.53 0)
 			(effects
 				(font
@@
 		)
 		(instances
-			(project ""
+			(project "mu"
 				(path "/0020f91a-50ae-478d-8303-55d8991d2d34"
 					(reference "J4")

Commit message: refactored following thoughts
Parts:
- removed J1: USB_C_Receptacle_USB2.0_16P, Connector_USB:USB_C_Receptacle_G-Switch_GT-USB-7010ASV, symbol Connector:USB_C_Receptacle_USB2.0_16P
- removed J2, J3: Conn_02x03_Odd_Even, Connector_PinHeader_1.00mm:PinHeader_2x03_P1.00mm_Vertical, symbol Connector_Generic:Conn_02x03_Odd_Even
- removed R12, R13: 10K, Resistor_SMD:R_0402_1005Metric, symbol Device:R
- removed R7, R8: 5.1K, Resistor_SMD:R_0402_1005Metric, symbol Device:R
- removed U7: USBLC6-2SC6, Package_TO_SOT_SMD:SOT-23-6, symbol Power_Protection:USBLC6-2SC6
- added C32: 100nF, Resistor_SMD:R_0402_1005Metric, symbol Device:C
- added J6: JTAG_SWD_10, Connector_IDC:IDC-Header_2x05_P2.54mm_Vertical, symbol Connector:Conn_ARM_JTAG_SWD_10
Connections:
- net PA+ is gone; now on net CAN_+: U1.18 (PA10/PA12)
- net PA- is gone; now on net CAN_-: U1.17 (PA9/PA11)
- net VBUS_RAW is gone; now on net 5V_LOGIC: D2.2
- net 3.3V_Dig: now also J6.1 (VTref)
- net 5V: now also C32.2
- net CAN_o-: now also J5.18; no longer J5.15
- net GND: now also J5.03, J5.04, C32.1, J6.3 (GND), J6.5 (GND), J6.9 (GNDDetect); no longer J5.01, J5.02, J5.13, J5.17, J5.18
- net NRST: now also J6.10 (~{RESET})
- net SWCLK: now also J6.4 (SWCLK/TCK)
- net SWDIO: now also J6.2 (SWDIO/TMS)
- net 5V_LOGIC: now reaches J5.05, J5.06
- net 5V_LOGIC: no longer J5.03, J5.04
- net Mode_sel: no longer names the net of U1.6 (PA0)
- new net 5v_SERVO: J5.01, J5.02
- new net NRST1: J5.09
- new net NRST2: J5.10
- new net NRST3: J5.11
- new net NRST4: J5.12
- new net NRST5: J5.13
- no-connect marks 12 -> 13
Other:
- note removed: "5v_logic not needed"
- note removed: "5v_servo not needed"
- note removed: "USB-C & mode select"
- moved on the sheet: C15, C30, J4, MOSFET1, U14

Commit message: huge
Parts:
- removed J6: JTAG_SWD_10, Connector_IDC:IDC-Header_2x05_P2.54mm_Vertical, symbol Connector:Conn_ARM_JTAG_SWD_10
- added J1: JTAG-10 PIN, Connector_IDC:IDC-Header_2x05_P2.54mm_Vertical, symbol Connector_Generic_MountingPin:Conn_01x10_MountingPin
Connections:
- net 3.3V_Dig: now also J1.7 (Pin_7), J1.8 (Pin_8)
- net GND: now also J1.5 (Pin_5), J1.6 (Pin_6)
- net NRST: now also J1.1 (Pin_1)
- net SWCLK: now also J1.2 (Pin_2)
- net SWDIO: now also J1.4 (Pin_4)
- no-connect marks 13 -> 15
Other:
- note added: "Connector_IDC:IDC-Header_2x05_P2.54mm_Vertical"
- note removed: "-"
