File: power.kicad_sch (KiCad schematic)
At the start: 25 parts, among them U7 MPM3650CGQW-P

Commit message: overhaul
Parts:
- added R24: 499kΩ, Resistor_SMD:R_0402_1005Metric, symbol Device:R
Connections:
- net vin: now also R24.2
- net at C34.1, C35.1, C36.1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: now also VR1.2 (IN_2)
- net at U7.16 (EN): now also R24.1
- no-connect marks 6 -> 7
Changed lines of the file:
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@@
+	)
+	(junction
+		(at 151.13 63.5)
+		(diameter 0)
+		(color 0 0 0 0)
 	)
 	(junction
@@
 	)
 	(junction
+		(at 64.77 86.36)
+		(diameter 0)
+		(color 0 0 0 0)
+	)
+	(junction
 		(at 123.19 63.5)
 		(diameter 0)
@@
 	)
 	(no_connect
+		(at 64.77 68.58)
+	)
+	(no_connect
 		(at 64.77 66.04)
 	)
@@
 	(wire
 		(pts
+			(xy 80.01 86.36) (xy 64.77 86.36)
+		)
+		(stroke
+			(width 0)
+			(type default)
+		)
+	)
+	(wire
+		(pts
 			(xy 129.54 55.88) (xy 135.89 55.88)
 		)
@@
 	(wire
 		(pts
+			(xy 60.96 71.12) (xy 60.96 69.85)
+		)
+		(stroke
+			(width 0)
+			(type default)
+		)
+	)
+	(wire
+		(pts
 			(xy 123.19 63.5) (xy 129.54 63.5)
 		)
@@
 	(wire
 		(pts
+			(xy 80.01 59.69) (xy 80.01 86.36)
+		)
+		(stroke
+			(width 0)
+			(type default)
+		)
+	)
+	(wire
+		(pts
+			(xy 60.96 62.23) (xy 60.96 59.69)
+		)
+		(stroke
+			(width 0)
+			(type default)
+		)
+	)
+	(wire
+		(pts
 			(xy 64.77 82.55) (xy 64.77 83.82)
 		)
@@
 	(wire
 		(pts
+			(xy 60.96 59.69) (xy 80.01 59.69)
+		)
+		(stroke
+			(width 0)
+			(type default)
+		)
+	)
+	(wire
+		(pts
 			(xy 58.42 86.36) (xy 52.07 86.36)
 		)
@@
 	(wire
 		(pts
+			(xy 64.77 71.12) (xy 60.96 71.12)
+		)
+		(stroke
+			(width 0)
+			(type default)
+		)
+	)
+	(wire
+		(pts
 			(xy 151.13 81.28) (xy 151.13 86.36)
 		)
@@
 		(pts
 			(xy 58.42 93.98) (xy 64.77 93.98)
+		)
+		(stroke
+			(width 0)
+			(type default)
+		)
+	)
+	(wire
+		(pts
+			(xy 151.13 63.5) (xy 151.13 66.04)
 		)
 		(stroke
@@
 					(unit 1)
 				)
+			)
+		)
+	)
+	(symbol
+		(lib_id "Device:R")
+		(at 60.96 66.04 180)
+		(unit 1)
+		(exclude_from_sim no)
+		(in_bom yes)
+		(on_board yes)
+		(dnp no)
+		(property "Reference" "R24"
+			(at 58.928 66.04 90)
+			(effects
+				(font
+					(size 1.27 1.27)
+				)
+			)
+		)
+		(property "Value" "499kΩ"
+			(at 60.96 66.04 90)
+			(effects
+				(font
+					(size 1.27 1.27)
+				)
+			)
+		)
+		(property "Footprint" "Resistor_SMD:R_0402_1005Metric"
+			(at 62.738 66.04 90)
+			(effects
+				(font
+					(size 1.27 1.27)
+				)
+				(hide yes)
+			)
+		)
+		(property "Datasheet" "~"
+			(at 60.96 66.04 0)
+			(effects
+				(font
+					(size 1.27 1.27)
+				)
+				(hide yes)
+			)
+		)
+		(property "Description" "Resistor"
+			(at 60.96 66.04 0)
+			(effects
+				(font
+					(size 1.27 1.27)
+				)
+				(hide yes)
+			)
+		)
+		(pin "2"
+		)
+		(pin "1"
+		)
+		(instances
+			(project "mu"
+				(path "/0020f91a-50ae-478d-8303-55d8991d2d34/9e4dd771-0c3b-45b5-a281-8d289f4a04ba"
+					(reference "R24")
+					(unit 1)
+				)

Commit message: ready for upload
Parts:
- removed R19: 750Ω, Resistor_SMD:R_0402_1005Metric, symbol Device:R
- removed R21: 200kΩ, Resistor_SMD:R_0402_1005Metric, symbol Device:R
- removed R22: 453kΩ, Resistor_SMD:R_0402_1005Metric, symbol Device:R
- removed R23: 49.9kΩ, Resistor_SMD:R_0402_1005Metric, symbol Device:R
- renumbered C34 to C32, C40 to C33, C41 to C34, C42 to C35, C43 to C37, C35 to C38, C37 to C39, C38 to C40, C39 to C41, C45 to C42, C44 to C43, C46 to C44, R13 to R16, R16 to R17, R5 to R18, R12 to R19, R24 to R20, R20 to R21, R18 to R22, U7 to U12
Connections:
- net GND: now also VR1.5 (ILIM)
- net at VR1.3 (EN/UV): now also C32.1, C36.1, C38.1, C39.1, C40.1, C41.1, C43.2, R17.2, U12.10 (OUT), U12.11 (OUT), U12.12 (OUT), U12.9 (OUT), VR1.1 (IN_1), VR1.2 (IN_2), VR1.6 (PGFB); no longer VR1.4 (PG)
- no-connect marks 7 -> 8

Commit message: ready for review the twost, nearly
Changed lines of the file:
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@@
+				)
+			)
+			(project "power"
+				(path "/add3bb49-27d0-4ece-b44a-27ddf0552b2e"
+					(reference "#PWR?")
+					(unit 1)
 				)
 			)
@@
 				)
 			)
+			(project "power"
+				(path "/add3bb49-27d0-4ece-b44a-27ddf0552b2e"
+					(reference "#PWR?")
+					(unit 1)
+				)
+			)
 		)
 	)
@@
 				)
 			)
+			(project "power"
+				(path "/add3bb49-27d0-4ece-b44a-27ddf0552b2e"
+					(reference "R?")
+					(unit 1)
+				)
+			)
 		)
 	)
@@
 				)
 			)
+			(project "power"
+				(path "/add3bb49-27d0-4ece-b44a-27ddf0552b2e"
+					(reference "C?")
+					(unit 1)
+				)
+			)
 		)
 	)
@@
 				)
 			)
+			(project "power"
+				(path "/add3bb49-27d0-4ece-b44a-27ddf0552b2e"
+					(reference "#PWR?")
+					(unit 1)
+				)
+			)
 		)
 	)
@@
 				)
 			)
+			(project "power"
+				(path "/add3bb49-27d0-4ece-b44a-27ddf0552b2e"
+					(reference "#PWR?")
+					(unit 1)
+				)
+			)
 		)
 	)
@@
 				)
 			)
+			(project "power"
+				(path "/add3bb49-27d0-4ece-b44a-27ddf0552b2e"
+					(reference "#PWR?")
+					(unit 1)
+				)
+			)
 		)
 	)
@@
 				)
 			)
+			(project "power"
+				(path "/add3bb49-27d0-4ece-b44a-27ddf0552b2e"
+					(reference "R?")
+					(unit 1)
+				)
+			)
 		)
 	)
@@
 				)
 			)
+			(project "power"
+				(path "/add3bb49-27d0-4ece-b44a-27ddf0552b2e"
+					(reference "C?")
+					(unit 1)
+				)
+			)
 		)
 	)
@@
 				)
 			)
+			(project "power"
+				(path "/add3bb49-27d0-4ece-b44a-27ddf0552b2e"
+					(reference "#PWR?")
+					(unit 1)
+				)
+			)
 		)
 	)
@@
 				)
 			)
+			(project "power"
+				(path "/add3bb49-27d0-4ece-b44a-27ddf0552b2e"
+					(reference "#PWR?")
+					(unit 1)
+				)
+			)
 		)
 	)
@@
 				)
 			)
+			(project "power"
+				(path "/add3bb49-27d0-4ece-b44a-27ddf0552b2e"
+					(reference "C?")
+					(unit 1)
+				)
+			)
 		)
 	)
@@
 				)
 			)
+			(project "power"
+				(path "/add3bb49-27d0-4ece-b44a-27ddf0552b2e"
+					(reference "C?")
+					(unit 1)
+				)
+			)
 		)
 	)
@@
 				)
 			)
+			(project "power"
+				(path "/add3bb49-27d0-4ece-b44a-27ddf0552b2e"
+					(reference "C?")
+					(unit 1)
+				)
+			)
 		)
 	)
@@
 				)
 			)
+			(project "power"
+				(path "/add3bb49-27d0-4ece-b44a-27ddf0552b2e"
+					(reference "#PWR?")
+					(unit 1)
+				)
+			)
 		)
 	)
@@
 		)
 		(property "Value" "33.2kΩ"
-			(at 147.32 81.28 90)
+			(at 147.32 78.994 90)
 			(effects
 				(font
@@
 				)
 			)
+			(project "power"
+				(path "/add3bb49-27d0-4ece-b44a-27ddf0552b2e"
+					(reference "R?")
+					(unit 1)
+				)
+			)
 		)
 	)
@@
 				)
 			)
+			(project "power"
+				(path "/add3bb49-27d0-4ece-b44a-27ddf0552b2e"
+					(reference "R?")
+					(unit 1)
+				)
+			)
 		)
 	)
@@
 				)
 			)
+			(project "power"
+				(path "/add3bb49-27d0-4ece-b44a-27ddf0552b2e"
+					(reference "C?")
+					(unit 1)
+				)
+			)
 		)
 	)
@@
 				)
 			)
+			(project "power"
+				(path "/add3bb49-27d0-4ece-b44a-27ddf0552b2e"
+					(reference "C?")
+					(unit 1)
+				)
+			)
 		)
 	)
@@
 				)
 			)
+			(project "power"
+				(path "/add3bb49-27d0-4ece-b44a-27ddf0552b2e"
+					(reference "#PWR?")
+					(unit 1)
+				)
+			)
 		)
 	)
@@
 				)
 			)
+			(project "power"
+				(path "/add3bb49-27d0-4ece-b44a-27ddf0552b2e"
+					(reference "R?")
+					(unit 1)
+				)
+			)
 		)
 	)
@@
 				)
 			)
+			(project "power"
+				(path "/add3bb49-27d0-4ece-b44a-27ddf0552b2e"
+					(reference "C?")
+					(unit 1)
+				)
+			)
 		)
 	)
@@
 				)
 			)
+			(project "power"
+				(path "/add3bb49-27d0-4ece-b44a-27ddf0552b2e"
+					(reference "C?")
+					(unit 1)
+				)
+			)
 		)
 	)
@@
 				)
 			)
+			(project "power"
+				(path "/add3bb49-27d0-4ece-b44a-27ddf0552b2e"
+					(reference "#PWR?")
+					(unit 1)
+				)
+			)
 		)
 	)
@@
 				)
 			)
+			(project "power"
+				(path "/add3bb49-27d0-4ece-b44a-27ddf0552b2e"
+					(reference "C?")
+					(unit 1)
+				)
+			)
 		)
 	)
@@
 				(path "/0020f91a-50ae-478d-8303-55d8991d2d34/9e4dd771-0c3b-45b5-a281-8d289f4a04ba"
 					(reference "C32")
+					(unit 1)
+				)
+			)
+			(project "power"
+				(path "/add3bb49-27d0-4ece-b44a-27ddf0552b2e"
+					(reference "C?")
 					(unit 1)
 				)
@@
 				)
 			)
+			(project "power"
+				(path "/add3bb49-27d0-4ece-b44a-27ddf0552b2e"
+					(reference "U?")
+					(unit 1)
+				)
+			)
 		)
 	)
@@
 				)
 			)
+			(project "power"
+				(path "/add3bb49-27d0-4ece-b44a-27ddf0552b2e"
+					(reference "R?")
+					(unit 1)
+				)
+			)
 		)
 	)
@@
 				)
 			)
+			(project "power"
+				(path "/add3bb49-27d0-4ece-b44a-27ddf0552b2e"
+					(reference "#PWR?")
+					(unit 1)
+				)
+			)
 		)
 	)
@@
 				)
 			)
+			(project "power"
+				(path "/add3bb49-27d0-4ece-b44a-27ddf0552b2e"
+					(reference "#PWR?")
+					(unit 1)
+				)
+			)
 		)
 	)
@@
 				)
 			)
+			(project "power"
+				(path "/add3bb49-27d0-4ece-b44a-27ddf0552b2e"
+					(reference "C?")
+					(unit 1)
+				)
+			)
 		)
 	)
@@
 				(path "/0020f91a-50ae-478d-8303-55d8991d2d34/9e4dd771-0c3b-45b5-a281-8d289f4a04ba"
 					(reference "R17")
+					(unit 1)
+				)
+			)
+			(project "power"
+				(path "/add3bb49-27d0-4ece-b44a-27ddf0552b2e"
+					(reference "R?")
 					(unit 1)
 				)
@@
 				)
 			)
+			(project "power"
+				(path "/add3bb49-27d0-4ece-b44a-27ddf0552b2e"
+					(reference "VR?")
+					(unit 1)
+				)
+			)
 		)
 	)
@@
 				)
 			)
-		)
-	)
+			(project "power"
+				(path "/add3bb49-27d0-4ece-b44a-27ddf0552b2e"
+					(reference "C?")
+					(unit 1)
+				)
+			)
+		)
+	)
+	(sheet_instances
+		(path "/"
+			(page "1")
+		)
+	)
+	(embedded_fonts no)
 )

Commit message: ready for review the twost, nearly, readout locked
Parts:
- renumbered C32 to C34, C33 to C35, C34 to C36, C35 to C37, C36 to C38, C37 to C39, C38 to C40, C39 to C41, C40 to C42, C41 to C43, C42 to C44, C43 to C45, C44 to C46, U12 to U11
Changed lines of the file:
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@@
 		(on_board yes)
 		(dnp no)
-		(property "Reference" "#PWR061"
+		(property "Reference" "#PWR055"
 			(at 58.42 76.2 0)
 			(effects
@@
 			(project "mu"
 				(path "/0020f91a-50ae-478d-8303-55d8991d2d34/9e4dd771-0c3b-45b5-a281-8d289f4a04ba"
-					(reference "#PWR061")
+					(reference "#PWR055")
 					(unit 1)
 				)
@@
 		(on_board yes)
 		(dnp no)
-		(property "Reference" "#PWR069"
+		(property "Reference" "#PWR063"
 			(at 187.96 86.36 0)
 			(effects
@@
 			(project "mu"
 				(path "/0020f91a-50ae-478d-8303-55d8991d2d34/9e4dd771-0c3b-45b5-a281-8d289f4a04ba"
-					(reference "#PWR069")
+					(reference "#PWR063")
 					(unit 1)
 				)
@@
 		(on_board yes)
 		(dnp no)
-		(property "Reference" "C34"
+		(property "Reference" "C36"
 			(at 56.388 92.202 0)
 			(effects
@@
 			(project "mu"
 				(path "/0020f91a-50ae-478d-8303-55d8991d2d34/9e4dd771-0c3b-45b5-a281-8d289f4a04ba"
-					(reference "C34")
+					(reference "C36")
 					(unit 1)
 				)
@@
 		(on_board yes)
 		(dnp no)
-		(property "Reference" "#PWR063"
+		(property "Reference" "#PWR057"
 			(at 114.3 91.44 0)
 			(effects
@@
 			(project "mu"
 				(path "/0020f91a-50ae-478d-8303-55d8991d2d34/9e4dd771-0c3b-45b5-a281-8d289f4a04ba"
-					(reference "#PWR063")
+					(reference "#PWR057")
 					(unit 1)
 				)
@@
 		(on_board yes)
 		(dnp no)
-		(property "Reference" "#PWR062"
+		(property "Reference" "#PWR056"
 			(at 64.77 100.33 0)
 			(effects
@@
 			(project "mu"
 				(path "/0020f91a-50ae-478d-8303-55d8991d2d34/9e4dd771-0c3b-45b5-a281-8d289f4a04ba"
-					(reference "#PWR062")
+					(reference "#PWR056")
 					(unit 1)
 				)
@@
 		(on_board yes)
 		(dnp no)
-		(property "Reference" "#PWR064"
+		(property "Reference" "#PWR058"
 			(at 124.46 78.74 0)
 			(effects
@@
 			(project "mu"
 				(path "/0020f91a-50ae-478d-8303-55d8991d2d34/9e4dd771-0c3b-45b5-a281-8d289f4a04ba"
-					(reference "#PWR064")
+					(reference "#PWR058")
 					(unit 1)
 				)
@@
 		(on_board yes)
 		(dnp no)
-		(property "Reference" "C33"
+		(property "Reference" "C35"
 			(at 50.038 92.202 0)
 			(effects
@@
 			(project "mu"
 				(path "/0020f91a-50ae-478d-8303-55d8991d2d34/9e4dd771-0c3b-45b5-a281-8d289f4a04ba"
-					(reference "C33")
+					(reference "C35")
 					(unit 1)
 				)
@@
 		(on_board yes)
 		(dnp no)
-		(property "Reference" "#PWR059"
+		(property "Reference" "#PWR053"
 			(at 55.88 111.76 0)
 			(effects
@@
 			(project ""
 				(path "/0020f91a-50ae-478d-8303-55d8991d2d34/9e4dd771-0c3b-45b5-a281-8d289f4a04ba"
-					(reference "#PWR059")
+					(reference "#PWR053")
 					(unit 1)
 				)
@@
 		(on_board yes)
 		(dnp no)
-		(property "Reference" "#PWR060"
+		(property "Reference" "#PWR054"
 			(at 63.5 111.76 0)
 			(effects
@@
 			(project "mu"
 				(path "/0020f91a-50ae-478d-8303-55d8991d2d34/9e4dd771-0c3b-45b5-a281-8d289f4a04ba"
-					(reference "#PWR060")
+					(reference "#PWR054")
 					(unit 1)
 				)
@@
 		(on_board yes)
 		(dnp no)
-		(property "Reference" "C36"
+		(property "Reference" "C38"
 			(at 114.808 61.722 0)
 			(effects
@@
 			(project "mu"
 				(path "/0020f91a-50ae-478d-8303-55d8991d2d34/9e4dd771-0c3b-45b5-a281-8d289f4a04ba"
-					(reference "C36")
+					(reference "C38")
 					(unit 1)
 				)
@@
 		(on_board yes)
 		(dnp no)
-		(property "Reference" "C41"
+		(property "Reference" "C43"
 			(at 140.208 61.722 0)
 			(effects
@@
 			(project "mu"
 				(path "/0020f91a-50ae-478d-8303-55d8991d2d34/9e4dd771-0c3b-45b5-a281-8d289f4a04ba"
-					(reference "C41")
+					(reference "C43")
 					(unit 1)
 				)
@@
 		(on_board yes)
 		(dnp no)
-		(property "Reference" "C44"
+		(property "Reference" "C46"
 			(at 185.928 61.722 0)
 			(effects
@@
 			(project "mu"
 				(path "/0020f91a-50ae-478d-8303-55d8991d2d34/9e4dd771-0c3b-45b5-a281-8d289f4a04ba"
-					(reference "C44")
+					(reference "C46")
 					(unit 1)
 				)
@@
 		(on_board yes)
 		(dnp no)
-		(property "Reference" "#PWR066"
+		(property "Reference" "#PWR060"
 			(at 137.16 76.2 0)
 			(effects
@@
 			(project "mu"
 				(path "/0020f91a-50ae-478d-8303-55d8991d2d34/9e4dd771-0c3b-45b5-a281-8d289f4a04ba"
-					(reference "#PWR066")
+					(reference "#PWR060")
 					(unit 1)
 				)
@@
 		(on_board yes)
 		(dnp no)
-		(property "Reference" "C42"
+		(property "Reference" "C44"
 			(at 145.288 90.678 0)
 			(effects
@@
 			(project "mu"
 				(path "/0020f91a-50ae-478d-8303-55d8991d2d34/9e4dd771-0c3b-45b5-a281-8d289f4a04ba"
-					(reference "C42")
+					(reference "C44")
 					(unit 1)
 				)
@@
 		(on_board yes)
 		(dnp no)
-		(property "Reference" "C43"
+		(property "Reference" "C45"
 			(at 145.542 57.658 0)
 			(effects
@@
 			(project "mu"
 				(path "/0020f91a-50ae-478d-8303-55d8991d2d34/9e4dd771-0c3b-45b5-a281-8d289f4a04ba"
-					(reference "C43")
+					(reference "C45")
 					(unit 1)
 				)
@@
 		(on_board yes)
 		(dnp no)
-		(property "Reference" "#PWR058"
+		(property "Reference" "#PWR052"
 			(at 35.56 77.47 0)
 			(effects
@@
 			(project "mu"
 				(path "/0020f91a-50ae-478d-8303-55d8991d2d34/9e4dd771-0c3b-45b5-a281-8d289f4a04ba"
-					(reference "#PWR058")
+					(reference "#PWR052")
 					(unit 1)
 				)
@@
 		(on_board yes)
 		(dnp no)
-		(property "Reference" "C39"
+		(property "Reference" "C41"
 			(at 127.508 61.722 0)
 			(effects
@@
 			(project "mu"
 				(path "/0020f91a-50ae-478d-8303-55d8991d2d34/9e4dd771-0c3b-45b5-a281-8d289f4a04ba"
-					(reference "C39")
+					(reference "C41")
 					(unit 1)
 				)
@@
 		(on_board yes)
 		(dnp no)
-		(property "Reference" "C38"
+		(property "Reference" "C40"
 			(at 121.158 61.722 0)
 			(effects
@@
 			(project "mu"
 				(path "/0020f91a-50ae-478d-8303-55d8991d2d34/9e4dd771-0c3b-45b5-a281-8d289f4a04ba"
-					(reference "C38")
+					(reference "C40")
 					(unit 1)
 				)
@@
 		(on_board yes)
 		(dnp no)
-		(property "Reference" "#PWR065"
+		(property "Reference" "#PWR059"
 			(at 135.89 48.26 0)
 			(effects
@@
 			(project "mu"
 				(path "/0020f91a-50ae-478d-8303-55d8991d2d34/9e4dd771-0c3b-45b5-a281-8d289f4a04ba"
-					(reference "#PWR065")
+					(reference "#PWR059")
 					(unit 1)
 				)
@@
 		(on_board yes)
 		(dnp no)
-		(property "Reference" "C37"
+		(property "Reference" "C39"
 			(at 116.332 74.422 0)
 			(effects
@@
 			(project "mu"
 				(path "/0020f91a-50ae-478d-8303-55d8991d2d34/9e4dd771-0c3b-45b5-a281-8d289f4a04ba"
-					(reference "C37")
+					(reference "C39")
 					(unit 1)
 				)
@@
 		(on_board yes)
 		(dnp no)
-		(property "Reference" "C32"
+		(property "Reference" "C34"
 			(at 38.862 66.548 0)
 			(effects
@@
 			(project ""
 				(path "/0020f91a-50ae-478d-8303-55d8991d2d34/9e4dd771-0c3b-45b5-a281-8d289f4a04ba"
-					(reference "C32")
+					(reference "C34")
 					(unit 1)
 				)
@@
 		(dnp no)
 		(fields_autoplaced yes)
-		(property "Reference" "U12"
+		(property "Reference" "U11"
 			(at 85.09 53.34 0)
 			(effects
@@
 			(project ""
 				(path "/0020f91a-50ae-478d-8303-55d8991d2d34/9e4dd771-0c3b-45b5-a281-8d289f4a04ba"
-					(reference "U12")
+					(reference "U11")
 					(unit 1)
 				)
@@
 		(on_board yes)
 		(dnp no)
-		(property "Reference" "#PWR067"
+		(property "Reference" "#PWR061"
 			(at 149.86 49.53 0)
 			(effects
@@
 			(project "mu"
 				(path "/0020f91a-50ae-478d-8303-55d8991d2d34/9e4dd771-0c3b-45b5-a281-8d289f4a04ba"
-					(reference "#PWR067")
+					(reference "#PWR061")
 					(unit 1)
 				)
@@
 		(on_board yes)
 		(dnp no)
-		(property "Reference" "#PWR068"
+		(property "Reference" "#PWR062"
 			(at 181.61 49.53 0)
 			(effects
@@
 			(project "mu"
 				(path "/0020f91a-50ae-478d-8303-55d8991d2d34/9e4dd771-0c3b-45b5-a281-8d289f4a04ba"
-					(reference "#PWR068")
+					(reference "#PWR062")
 					(unit 1)
 				)
@@
 		(on_board yes)
 		(dnp no)
-		(property "Reference" "C35"
+		(property "Reference" "C37"
 			(at 62.738 92.202 0)
 			(effects
@@
 			(project "mu"
 				(path "/0020f91a-50ae-478d-8303-55d8991d2d34/9e4dd771-0c3b-45b5-a281-8d289f4a04ba"
-					(reference "C35")
+					(reference "C37")
 					(unit 1)
 				)
@@
 		(on_board yes)
 		(dnp no)
-		(property "Reference" "C40"
+		(property "Reference" "C42"
 			(at 133.858 61.722 0)
 			(effects
@@
 			(project "mu"
 				(path "/0020f91a-50ae-478d-8303-55d8991d2d34/9e4dd771-0c3b-45b5-a281-8d289f4a04ba"
-					(reference "C40")
-					(unit 1)
-				)
+					(reference "C42")
+					(unit 1)
+				)
