File: power.kicad_sch (KiCad schematic)
At the start: 22 parts, among them U11 MPM3650CGQW-P

Commit message: hardware done
Parts:
- removed R18, R19: 0Ω, Resistor_SMD:R_0402_1005Metric, symbol Device:R
- removed R20: 499kΩ, Resistor_SMD:R_0402_1005Metric, symbol Device:R
- C36, C37, C40, C41, C42, C43, C46: footprint Capacitor_SMD:C_0402_1005Metric -> Capacitor_SMD:C_0603_1608Metric
Connections:
- net GND is gone; now on net AGND: C35.1, C36.1, C37.1, C38.2, C40.2, C41.2, C42.2, C43.2, C44.1, C45.1, C46.2, R22.2, U11.1 (PGND), U11.2 (PGND), U11.24 (PGND), U11.3 (PGND), U11.4 (PGND), U11.5 (PGND), VR1.11 (EXP), VR1.5 (ILIM), VR1.8 (GND)
- net vin: now also U11.16 (EN)
- net at C34.2, R16.2, R17.1: now also U11.17 (FB)
Other:
- moved on the sheet: C39
